Commit message: Debugging ustbot urdf file for correct implementation in Gazebo

File: src/Simulation/Descriptions/ustbot_description/urdf/ustbot.urdf (robot description, URDF)
Before this commit: robot ustbot, 29 links, 28 joints
Links:
- removed link arm_base_link
- removed link bicep_link
- removed link bracelet_link
- removed link forearm_link
- removed link shoulder_link
- removed link spherical_wrist_1_link
- removed link spherical_wrist_2_link
Joints:
- removed joint arm_base_joint
- removed joint bicep_joint
- removed joint bracelet_joint
- removed joint forearm_joint
- removed joint shoulder_joint
- removed joint spherical_wrist_2_joint
- removed joint spherocal_wrist_1_joint
