Commit message: Adding diff drive controllers for simulation

File: src/Simulation/Descriptions/ustbot_description/urdf/ustbot.urdf.xacro (robot description, xacro)
@@ -4,5 +4,15 @@
      For more information, please see http://wiki.ros.org/sw_urdf_exporter -->
 <robot
-  name="ustbot">
+  name="ustbot"
+  xmlns:xacro="http://ros.org/wiki/xacro">
+  <xacro:include filename="$(find ustbot_description)/urdf/ustbot.gazebo.xacro"/>
+  <!-- Used for fixing robot to Gazebo 'base_link' -->
+  <!--
+  <link name="world"/>
+  <joint name="fixed" type="fixed">
+    <parent link="world"/>
+    <child link="link1"/>
+  </joint>
+  -->
   <link  name="base_footprint"/>
   <joint name="base_joint" type="fixed">
@@ -15,4 +25,5 @@
       rpy="0 0 0"/>
   </joint>
+  <!-- ******************************************** -->
   <link name="base_link">
     <inertial>
@@ -109,4 +120,13 @@
       velocity="1000" />
   </joint>
+  <transmission name="left_wheelhub_transmission">
+    <type>transmission_interface/SimpleTransmission</type>
+    <joint name="left_wheelhub_joint">
+      <hardwareInterface>hardware_interface/VelocityJointInterface</hardwareInterface>
+    </joint>
+    <actuator name="left_wheelhub_actuator">
+      <hardwareInterface>VelocityJointInterface</hardwareInterface>
+    </actuator>
+  </transmission>
   <link name="right_wheelhub_link">
     <inertial>
@@ -164,4 +184,13 @@
       velocity="1000" />
   </joint>
+  <transmission name="right_wheelhub_transmission">
+    <type>transmission_interface/SimpleTransmission</type>
+    <joint name="right_wheelhub_joint">
+      <hardwareInterface>hardware_interface/VelocityJointInterface</hardwareInterface>
+    </joint>
+    <actuator name="right_wheelhub_actuator">
+      <hardwareInterface>VelocityJointInterface</hardwareInterface>
+    </actuator>
+  </transmission>
   <link name="left_front_universal_link">
     <inertial>

Commit message: Improving diff controler by changing the correct wheel separation

File: src/Simulation/Descriptions/ustbot_description/urdf/ustbot.urdf.xacro (robot description, xacro)
@@ -235,5 +235,5 @@
     </collision>
   </link>
-  <joint name="left_front_universal_joint" type="fixed">
+  <joint name="left_front_universal_joint" type="continuous">
     <origin
       xyz="0.32 0.199 0.012"
@@ -290,5 +290,5 @@
     </collision>
   </link>
-  <joint name="left_front_universalWheel_joint" type="fixed">
+  <joint name="left_front_universalWheel_joint" type="continuous">
     <origin
       xyz="-0.035 0 0.052"
@@ -345,5 +345,5 @@
     </collision>
   </link>
-  <joint name="left_back_universal_joint" type="fixed">
+  <joint name="left_back_universal_joint" type="continuous">
     <origin
       xyz="-0.319 0.199 0.012"
@@ -400,5 +400,5 @@
     </collision>
   </link>
-  <joint name="left_back_universalWheel_joint" type="fixed">
+  <joint name="left_back_universalWheel_joint" type="continuous">
     <origin
       xyz="-0.035 0 0.052"
@@ -455,5 +455,5 @@
     </collision>
   </link>
-  <joint name="right_back_universal_joint" type="fixed">
+  <joint name="right_back_universal_joint" type="continuous">
     <origin
       xyz="-0.32 -0.199 0.012"
@@ -510,5 +510,5 @@
     </collision>
   </link>
-  <joint name="right_back_universalWheel_joint" type="fixed">
+  <joint name="right_back_universalWheel_joint" type="continuous">
     <origin
       xyz="-0.035 0 0.052"
@@ -565,5 +565,5 @@
     </collision>
   </link>
-  <joint name="right_front_universal_joint" type="fixed">
+  <joint name="right_front_universal_joint" type="continuous">
     <origin
       xyz="0.319 -0.199 0.012"
@@ -620,5 +620,5 @@
     </collision>
   </link>
-  <joint name="right_front_universalWheel_joint" type="fixed">
+  <joint name="right_front_universalWheel_joint" type="continuous">
     <origin
       xyz="-0.035 0 0.052"
