Commit message: Fixing URDF file and adding including necessary controllers for publishing joint states

File: src/Simulation/Descriptions/ustbot_description/urdf/ustbot.gazebo.xacro (robot description, xacro)
@@ -9,6 +9,6 @@
   </gazebo>
   <gazebo reference="left_front_universalWheel_link">
-    <mu1>0.1</mu1>
-    <mu2>0.1</mu2>
+    <mu1>0.01</mu1>
+    <mu2>0.01</mu2>
     <kp>500000.0</kp>
     <kd>10.0</kd>
@@ -19,6 +19,6 @@
   </gazebo>
   <gazebo reference="right_front_universalWheel_link">
-    <mu1>0.1</mu1>
-    <mu2>0.1</mu2>
+    <mu1>0.01</mu1>
+    <mu2>0.01</mu2>
     <kp>500000.0</kp>
     <kd>10.0</kd>
@@ -29,8 +29,8 @@
   </gazebo>
   <gazebo reference="left_back_universalWheel_link">
-    <mu1>0.1</mu1>
-    <mu2>0.1</mu2>
+    <mu1>0.01</mu1>
+    <mu2>0.01</mu2>
     <kp>500000.0</kp>
-    <kd>10.0</kd>
+    <kd>100.0</kd>
     <minDepth>0.001</minDepth>
     <maxVel>0.1</maxVel>
@@ -39,8 +39,8 @@
   </gazebo>
   <gazebo reference="right_back_universalWheel_link">
-    <mu1>0.1</mu1>
-    <mu2>0.1</mu2>
+    <mu1>0.01</mu1>
+    <mu2>0.01</mu2>
     <kp>500000.0</kp>
-    <kd>10.0</kd>
+    <kd>100.0</kd>
     <minDepth>0.001</minDepth>
     <maxVel>0.1</maxVel>

File: src/Simulation/Descriptions/ustbot_description/urdf/ustbot.urdf.xacro (robot description, xacro)
@@ -26,4 +26,5 @@
   </joint>
   <!-- ******************************************** -->
+  <!-- ********** Driven Wheels Section ********** -->
   <link name="base_link">
     <inertial>
@@ -104,7 +105,7 @@
     </collision>
   </link>
-  <joint name="left_wheelhub_joint" type="revolute">
-    <origin
-      xyz="0 0.19 0"
+  <joint name="left_wheelhub_joint" type="continuous">
+    <origin
+      xyz="0 0.19 0.005"
       rpy="-1.5708 0 0" />
     <parent
@@ -113,5 +114,5 @@
       link="left_wheelhub_link" />
     <axis
-      xyz="0 0 -1" />
+      xyz="0 0 1" />
     <limit
       lower="-10000"
@@ -168,7 +169,7 @@
     </collision>
   </link>
-  <joint name="right_wheelhub_joint" type="revolute">
-    <origin
-      xyz="0 -0.19 0"
+  <joint name="right_wheelhub_joint" type="continuous">
+    <origin
+      xyz="0 -0.19 0.005"
       rpy="-1.5708 0 0" />
     <parent
@@ -193,4 +194,6 @@
     </actuator>
   </transmission>
+  <!-- ******************************************** -->
+  <!-- *******Suport Wheels Section******* -->
   <link name="left_front_universal_link">
     <inertial>
@@ -232,5 +235,5 @@
     </collision>
   </link>
-  <joint name="left_front_universal_joint" type="revolute">
+  <joint name="left_front_universal_joint" type="fixed">
     <origin
       xyz="0.32 0.199 0.012"
@@ -287,5 +290,5 @@
     </collision>
   </link>
-  <joint name="left_front_universalWheel_joint" type="revolute">
+  <joint name="left_front_universalWheel_joint" type="fixed">
     <origin
       xyz="-0.035 0 0.052"
@@ -342,5 +345,5 @@
     </collision>
   </link>
-  <joint name="left_back_universal_joint" type="revolute">
+  <joint name="left_back_universal_joint" type="fixed">
     <origin
       xyz="-0.319 0.199 0.012"
@@ -397,5 +400,5 @@
     </collision>
   </link>
-  <joint name="left_back_universalWheel_joint" type="revolute">
+  <joint name="left_back_universalWheel_joint" type="fixed">
     <origin
       xyz="-0.035 0 0.052"
@@ -452,5 +455,5 @@
     </collision>
   </link>
-  <joint name="right_back_universal_joint" type="revolute">
+  <joint name="right_back_universal_joint" type="fixed">
     <origin
       xyz="-0.32 -0.199 0.012"
@@ -507,5 +510,5 @@
     </collision>
   </link>
-  <joint name="right_back_universalWheel_joint" type="revolute">
+  <joint name="right_back_universalWheel_joint" type="fixed">
     <origin
       xyz="-0.035 0 0.052"
@@ -562,5 +565,5 @@
     </collision>
   </link>
-  <joint name="right_front_universal_joint" type="revolute">
+  <joint name="right_front_universal_joint" type="fixed">
     <origin
       xyz="0.319 -0.199 0.012"
@@ -617,5 +620,5 @@
     </collision>
   </link>
-  <joint name="right_front_universalWheel_joint" type="revolute">
+  <joint name="right_front_universalWheel_joint" type="fixed">
     <origin
       xyz="-0.035 0 0.052"
@@ -633,4 +636,393 @@
       velocity="1000" />
   </joint>
+  <!-- ******************************************** -->
+  <!--
+  <link name="arm_base_link">
+    <inertial>
+      <origin
+        xyz="-0.000711712698347439 0.000106262049453287 0.0781492762008092"
+        rpy="0 0 0" />
+      <mass
+        value="1.06209181455169" />
+      <inertia
+        ixx="0.00275577215631917"
+        ixy="-1.14162264322392E-07"
+        ixz="-2.81022161469274E-05"
+        iyy="0.00277993758214866"
+        iyz="-1.83036413267701E-06"
+        izz="0.00115303923244668" />
+    </inertial>
+    <visual>
+      <origin
+        xyz="0 0 0"
+        rpy="0 0 0" />
+      <geometry>
+        <mesh
+          filename="package://ustbot_description/meshes/arm_base_link.STL" />
+      </geometry>
+      <material
+        name="">
+        <color
+          rgba="0.792156862745098 0.819607843137255 0.933333333333333 1" />
+      </material>
+    </visual>
+    <collision>
+      <origin
+        xyz="0 0 0"
+        rpy="0 0 0" />
+      <geometry>
+        <mesh
+          filename="package://ustbot_description/meshes/arm_base_link.STL" />
+      </geometry>
+    </collision>
+  </link>
+  <joint name="arm_base_joint" type="fixed">
+    <origin
+      xyz="0.235 0 0.6535"
+      rpy="0 0 0" />
+    <parent
+      link="base_link" />
+    <child
+      link="arm_base_link" />
+    <axis
+      xyz="0 0 0" />
+    <limit
+      lower="-10000"
+      upper="10000"
+      effort="1000"
+      velocity="1000" />
+  </joint>
+  <link name="shoulder_link">
+    <inertial>
+      <origin
+        xyz="-0.0840018720035909 -0.208802974838312 -0.872375327554249"
+        rpy="0 0 0" />
+      <mass
+        value="0.508433094676871" />
+      <inertia
+        ixx="0.000700265716566138"
+        ixy="1.885546538717E-08"
+        ixz="2.09523894060598E-08"
+        iyy="0.00082734360816898"
+        iyz="-7.35265759047621E-05"
+        izz="0.000489245693764828" />
+    </inertial>
+    <visual>
+      <origin
+        xyz="0 0 0"
+        rpy="0 0 0" />
+      <geometry>
+        <mesh
+          filename="package://ustbot_description/meshes/shoulder_link.STL" />
+      </geometry>
+      <material
+        name="">
+        <color
+          rgba="0.792156862745098 0.819607843137255 0.933333333333333 1" />
+      </material>
+    </visual>
+    <collision>
+      <origin
+        xyz="0 0 0"
+        rpy="0 0 0" />
+      <geometry>
+        <mesh
+          filename="package://ustbot_description/meshes/shoulder_link.STL" />
+      </geometry>
+    </collision>
+  </link>
+  <joint name="shoulder_joint" type="revolute">
+    <origin
+      xyz="0.084 -0.199 -0.6415"
+      rpy="-3.1416 0 0" />
+    <parent
+      link="arm_base_link" />
+    <child
+      link="shoulder_link" />
+    <axis
+      xyz="0 0 -1" />
+    <limit
+      lower="-10000"
+      upper="10000"
+      effort="1000"
+      velocity="1000" />
+  </joint>
+  <link name="bicep_link">
+    <inertial>
+      <origin
+        xyz="-1.44667187100544E-05 -0.209035829145565 -0.00477389800841804"
+        rpy="0 0 0" />
+      <mass
+        value="0.492119196746743" />
+      <inertia
+        ixx="0.00279565951071861"
+        ixy="-1.41208694363429E-07"
+        ixz="7.44180893992196E-08"
+        iyy="0.000309455115357151"
+        iyz="8.09747787651918E-08"
+        izz="0.00299614904881225" />
+    </inertial>
+    <visual>
+      <origin
+        xyz="0 0 0"
+        rpy="0 0 0" />
+      <geometry>
+        <mesh
+          filename="package://ustbot_description/meshes/bicep_link.STL" />
+      </geometry>
+      <material
+        name="">
+        <color
+          rgba="0.792156862745098 0.819607843137255 0.933333333333333 1" />
+      </material>
+    </visual>
+    <collision>
+      <origin
+        xyz="0 0 0"
+        rpy="0 0 0" />
+      <geometry>
+        <mesh
+          filename="package://ustbot_description/meshes/bicep_link.STL" />
+      </geometry>
+    </collision>
+  </link>
+  <joint name="bicep_joint" type="revolute">
+    <origin
+      xyz="-0.084 -0.1792 -0.9263"
+      rpy="1.5708 0 0" />
+    <parent
+      link="shoulder_link" />
+    <child
+      link="bicep_link" />
+    <axis
+      xyz="0 0 -1" />
+    <limit
+      lower="-10000"
+      upper="10000"
+      effort="1000"
+      velocity="1000" />
+  </joint>
+  <link name="forearm_link">
+    <inertial>
+      <origin
+        xyz="-4.16309103992707E-06 0.0799449656387601 -0.00673657663584737"
+        rpy="0 0 0" />
+      <mass
+        value="0.109261809919368" />
+      <inertia
+        ixx="0.00039446074043438"
+        ixy="-9.56510853411388E-08"
+        ixz="-8.46662670511317E-09"
+        iyy="0.000112362718424169"
+        iyz="-5.78354109274912E-05"
+        izz="0.000423666778381865" />
+    </inertial>
+    <visual>
+      <origin
+        xyz="0 0 0"
+        rpy="0 0 0" />
+      <geometry>
+        <mesh
+          filename="package://ustbot_description/meshes/forearm_link.STL" />
+      </geometry>
+      <material
+        name="">
+        <color
+          rgba="0.792156862745098 0.819607843137255 0.933333333333333 1" />
+      </material>
+    </visual>
+    <collision>
+      <origin
+        xyz="0 0 0"
+        rpy="0 0 0" />
+      <geometry>
+        <mesh
+          filename="package://ustbot_description/meshes/forearm_link.STL" />
+      </geometry>
+    </collision>
+  </link>
+  <joint name="forearm_joint" type="revolute">
+    <origin
+      xyz="0 -0.41 0.02885"
+      rpy="3.1416 0 0" />
+    <parent
+      link="bicep_link" />
+    <child
+      link="forearm_link" />
+    <axis
+      xyz="0 0 1" />
+    <limit
+      lower="-10000"
+      upper="10000"
+      effort="1000"
+      velocity="1000" />
+  </joint>
+  <link name="spherical_wrist_1_link">
+    <inertial>
+      <origin
+        xyz="-1.33966470524938E-05 0.0134681682665654 0.0569185239491965"
+        rpy="0 0 0" />
+      <mass
+        value="0.0607181356041409" />
+      <inertia
+        ixx="0.000138166287093796"
+        ixy="-1.36300678114682E-08"
+        ixz="-4.46917368595719E-08"
+        iyy="0.000140550901694903"
+        iyz="-2.20908893258633E-05"
+        izz="5.89037344032269E-05" />
+    </inertial>
+    <visual>
+      <origin
+        xyz="0 0 0"
+        rpy="0 0 0" />
+      <geometry>
+        <mesh
+          filename="package://ustbot_description/meshes/spherical_wrist_1_link.STL" />
+      </geometry>
+      <material
+        name="">
+        <color
+          rgba="0.792156862745098 0.819607843137255 0.933333333333333 1" />
+      </material>
+    </visual>
+    <collision>
+      <origin
+        xyz="0 0 0"
+        rpy="0 0 0" />
+      <geometry>
+        <mesh
+          filename="package://ustbot_description/meshes/spherical_wrist_1_link.STL" />
+      </geometry>
+    </collision>
+  </link>
+  <joint name="spherocal_wrist_1_joint" type="revolute">
+    <origin
+      xyz="0 0.2209 0.00805"
+      rpy="-1.5708 0 0" />
+    <parent
+      link="forearm_link" />
+    <child
+      link="spherical_wrist_1_link" />
+    <axis
+      xyz="0 0 1" />
+    <limit
+      lower="-10000"
+      upper="10000"
+      effort="1000"
+      velocity="1000" />
+  </joint>
+  <link name="spherical_wrist_2_link">
+    <inertial>
+      <origin
+        xyz="-7.14531001405616E-06 -0.0467740828401713 -0.00106495389643069"
+        rpy="0 0 0" />
+      <mass
+        value="0.0606982648446486" />
+      <inertia
+        ixx="0.000151586780132747"
+        ixy="-1.27452373879111E-08"
+        ixz="5.33427994049047E-09"
+        iyy="6.22322674674967E-05"
+        iyz="3.01646882784132E-05"
+        izz="0.000150621081679687" />
+    </inertial>
+    <visual>
+      <origin
+        xyz="0 0 0"
+        rpy="0 0 0" />
+      <geometry>
+        <mesh
+          filename="package://ustbot_description/meshes/spherical_wrist_2_link.STL" />
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
Commit message: ustbot low poly demo

File: src/Simulation/Descriptions/ustbot_description/urdf/ustbot.gazebo.xacro (robot description, xacro)
@@ -1,180 +1,113 @@
-<?xml version="1.0"?>
-<robot name="ustbot_sim" xmlns:xacro="http://ros.org/wiki/xacro">
-  <!--
-  <xacro:arg name="laser_visual" default="false"/>
-  <xacro:arg name="imu_visual"   default="false"/>
-  -->
-  <gazebo reference="base_link">
-    <material>Gazebo/DarkGrey</material>
-  </gazebo>
-  <gazebo reference="left_front_universalWheel_link">
-    <mu1>0.01</mu1>
-    <mu2>0.01</mu2>
-    <kp>500000.0</kp>
-    <kd>10.0</kd>
-    <minDepth>0.001</minDepth>
-    <maxVel>0.1</maxVel>
-    <fdir1>1 0 0</fdir1>
-    <material>Gazebo/FlatBlack</material>
-  </gazebo>
-  <gazebo reference="right_front_universalWheel_link">
-    <mu1>0.01</mu1>
-    <mu2>0.01</mu2>
-    <kp>500000.0</kp>
-    <kd>10.0</kd>
-    <minDepth>0.001</minDepth>
-    <maxVel>0.1</maxVel>
-    <fdir1>1 0 0</fdir1>
-    <material>Gazebo/FlatBlack</material>
-  </gazebo>
-  <gazebo reference="left_back_universalWheel_link">
-    <mu1>0.01</mu1>
-    <mu2>0.01</mu2>
-    <kp>500000.0</kp>
-    <kd>100.0</kd>
-    <minDepth>0.001</minDepth>
-    <maxVel>0.1</maxVel>
-    <fdir1>1 0 0</fdir1>
-    <material>Gazebo/FlatBlack</material>
-  </gazebo>
-  <gazebo reference="right_back_universalWheel_link">
-    <mu1>0.01</mu1>
-    <mu2>0.01</mu2>
-    <kp>500000.0</kp>
-    <kd>100.0</kd>
-    <minDepth>0.001</minDepth>
-    <maxVel>0.1</maxVel>
-    <fdir1>1 0 0</fdir1>
-    <material>Gazebo/FlatBlack</material>
-  </gazebo>
-  <gazebo reference="left_wheelhub_link">
-    <mu1>0.1</mu1>
-    <mu2>0.1</mu2>
-    <kp>1000000.0</kp>
-    <kd>100.0</kd>
-    <minDepth>0.001</minDepth>
-    <maxVel>1.0</maxVel>
-    <material>Gazebo/FlatBlack</material>
-  </gazebo>
-  <gazebo reference="right_wheelhub_link">
-    <mu1>0.1</mu1>
-    <mu2>0.1</mu2>
-    <kp>1000000.0</kp>
-    <kd>100.0</kd>
-    <minDepth>0.001</minDepth>
-    <maxVel>1.0</maxVel>
-    <material>Gazebo/FlatBlack</material>
-  </gazebo>
-  <gazebo>
-    <plugin name="gazebo_ros_control" filename="libgazebo_ros_control.so">
-    </plugin>
-  </gazebo>
-  <!--
-  <gazebo>
-    <plugin name="ustbot_controller" filename="libgazebo_ros_diff_drive.so">
-      <commandTopic>cmd_vel</commandTopic>
-      <odometryTopic>odom</odometryTopic>
-      <odometryFrame>odom</odometryFrame>
-      <odometrySource>world</odometrySource>
-      <publishOdomTF>true</publishOdomTF>
-      <robotBaseFrame>base_footprint</robotBaseFrame>
-      <publishWheelTF>false</publishWheelTF>
-      <publishTf>true</publishTf>
-      <publishWheelJointState>true</publishWheelJointState>
-      <legacyMode>false</legacyMode>
-      <updateRate>30</updateRate>
-      <leftJoint>wheel_left_joint</leftJoint>
-      <rightJoint>wheel_right_joint</rightJoint>
-      <wheelSeparation>0.45</wheelSeparation>
-      <wheelDiameter>0.165</wheelDiameter>
-      <wheelAcceleration>1</wheelAcceleration>
-      <wheelTorque>10</wheelTorque>
-      <rosDebugLevel>na</rosDebugLevel>
-    </plugin>
-  </gazebo>
-  -->
-  <!--
-  <gazebo>
-    <plugin name="ustbot_controller" filename="libgazebo_ros_diff_drive.so">
-      <commandTopic>cmd_vel</commandTopic>
-      <odometryTopic>odom</odometryTopic>
-      <odometryFrame>odom</odometryFrame>
-      <odometrySource>world</odometrySource>
-      <publishOdomTF>true</publishOdomTF>
-      <robotBaseFrame>base_footprint</robotBaseFrame>
-      <publishWheelTF>false</publishWheelTF>
-      <publishTf>true</publishTf>
-      <publishWheelJointState>true</publishWheelJointState>
-      <legacyMode>false</legacyMode>
-      <updateRate>30</updateRate>
-      <leftJoint>wheel_left_joint</leftJoint>
-      <rightJoint>wheel_right_joint</rightJoint>
-      <wheelSeparation>0.160</wheelSeparation>
-      <wheelDiameter>0.066</wheelDiameter>
-      <wheelAcceleration>1</wheelAcceleration>
-      <wheelTorque>10</wheelTorque>
-      <rosDebugLevel>na</rosDebugLevel>
-    </plugin>
-  </gazebo>
-  <gazebo>
-    <plugin name="imu_plugin" filename="libgazebo_ros_imu.so">
-      <alwaysOn>true</alwaysOn>
-      <bodyName>imu_link</bodyName>
-      <frameName>imu_link</frameName>
-      <topicName>imu</topicName>
-      <serviceName>imu_service</serviceName>
-      <gaussianNoise>0.0</gaussianNoise>
-      <updateRate>0</updateRate>
-      <imu>
-        <noise>
-          <type>gaussian</type>
-          <rate>
-            <mean>0.0</mean>
-            <stddev>2e-4</stddev>
-            <bias_mean>0.0000075</bias_mean>
-            <bias_stddev>0.0000008</bias_stddev>
-          </rate>
-          <accel>
-            <mean>0.0</mean>
-            <stddev>1.7e-2</stddev>
-            <bias_mean>0.1</bias_mean>
-            <bias_stddev>0.001</bias_stddev>
-          </accel>
-        </noise>
-      </imu>
-    </plugin>
-  </gazebo>
-  <gazebo reference="base_scan">
-    <material>Gazebo/FlatBlack</material>
-    <sensor type="ray" name="lds_lfcd_sensor">
-      <pose>0 0 0 0 0 0</pose>
-      <visualize>$(arg laser_visual)</visualize>
-      <update_rate>5</update_rate>
-      <ray>
-        <scan>
-          <horizontal>
-            <samples>360</samples>
-            <resolution>1</resolution>
-            <min_angle>0.0</min_angle>
-            <max_angle>6.28319</max_angle>
-          </horizontal>
-        </scan>
-        <range>
-          <min>0.120</min>
-          <max>3.5</max>
-          <resolution>0.015</resolution>
-        </range>
-        <noise>
-          <type>gaussian</type>
-          <mean>0.0</mean>
-          <stddev>0.01</stddev>
-        </noise>
-      </ray>
-      <plugin name="gazebo_ros_lds_lfcd_controller" filename="libgazebo_ros_laser.so">
-        <topicName>scan</topicName>
-        <frameName>base_scan</frameName>
-      </plugin>
-    </sensor>
-  </gazebo>
-  -->
+<?xml version="1.0" ?>
+<robot name="ustbot" xmlns:xacro="http://www.ros.org/wiki/xacro" >
+<xacro:property name="body_color" value="Gazebo/Silver" />
+<!--
+<gazebo>
+  <plugin name="gazebo_ros_control" filename="libgazebo_ros_control.so">
+  </plugin>
+</gazebo>
+-->
+<gazebo>
+  <plugin name="ustbot_controller" filename="libgazebo_ros_diff_drive.so">
+    <commandTopic>cmd_vel</commandTopic>
+    <odometryTopic>odom</odometryTopic>
+    <odometryFrame>odom</odometryFrame>
+    <odometrySource>world</odometrySource>
+    <publishOdomTF>true</publishOdomTF>
+    <robotBaseFrame>base_footprint</robotBaseFrame>
+    <publishWheelTF>false</publishWheelTF>
+    <publishTf>true</publishTf>
+    <publishWheelJointState>true</publishWheelJointState>
+    <legacyMode>false</legacyMode>
+    <updateRate>30</updateRate>
+    <leftJoint>wheel_left_joint</leftJoint>
+    <rightJoint>wheel_right_joint</rightJoint>
+    <wheelSeparation>0.45</wheelSeparation>
+    <wheelDiameter>0.165</wheelDiameter>
+    <wheelAcceleration>1</wheelAcceleration>
+    <wheelTorque>100</wheelTorque>
+    <rosDebugLevel>na</rosDebugLevel>
+  </plugin>
+</gazebo>
+<gazebo reference="base_link">
+  <material>${body_color}</material>
+  <mu1>0.1</mu1>
+  <mu2>0.1</mu2>
+  <selfCollide>true</selfCollide>
+  <gravity>true</gravity>
+</gazebo>
+<gazebo reference="wheel_right">
+  <material>${body_color}</material>
+  <mu1>3500</mu1>
+  <mu2>3500</mu2>
+  <selfCollide>true</selfCollide>
+</gazebo>
+<gazebo reference="wheel_left">
+  <material>${body_color}</material>
+  <mu1>3500</mu1>
+  <mu2>3500</mu2>
+  <selfCollide>true</selfCollide>
+</gazebo>
+<!--
+<gazebo reference="ultrasonic_front_right">
+  <material>${body_color}</material>
+  <mu1>0.2</mu1>
+  <mu2>0.2</mu2>
+  <selfCollide>true</selfCollide>
+</gazebo>
+<gazebo reference="ultrasonic_front_left">
+  <material>${body_color}</material>
+  <mu1>0.2</mu1>
+  <mu2>0.2</mu2>
+  <selfCollide>true</selfCollide>
+</gazebo>
+<gazebo reference="ultrasonic_left_left">
+  <material>${body_color}</material>
+  <mu1>0.2</mu1>
+  <mu2>0.2</mu2>
+  <selfCollide>true</selfCollide>
+</gazebo>
+<gazebo reference="ultrasonic_left_right">
+  <material>${body_color}</material>
+  <mu1>0.2</mu1>
+  <mu2>0.2</mu2>
+  <selfCollide>true</selfCollide>
+</gazebo>
+<gazebo reference="ultrasonic_back_left">
+  <material>${body_color}</material>
+  <mu1>0.2</mu1>
+  <mu2>0.2</mu2>
+  <selfCollide>true</selfCollide>
+</gazebo>
+<gazebo reference="ultrasonic_back_right">
+  <material>${body_color}</material>
+  <mu1>0.2</mu1>
+  <mu2>0.2</mu2>
+  <selfCollide>true</selfCollide>
+</gazebo>
+<gazebo reference="ultrasonic_right_left">
+  <material>${body_color}</material>
+  <mu1>0.2</mu1>
+  <mu2>0.2</mu2>
+  <selfCollide>true</selfCollide>
+</gazebo>
+<gazebo reference="ultrasonic_right_right">
+  <material>${body_color}</material>
+  <mu1>0.2</mu1>
+  <mu2>0.2</mu2>
+  <selfCollide>true</selfCollide>
+</gazebo>
+<gazebo reference="lidar_front">
+  <material>${body_color}</material>
+  <mu1>0.2</mu1>
+  <mu2>0.2</mu2>
+  <selfCollide>true</selfCollide>
+</gazebo>
+<gazebo reference="lidar_back">
+  <material>${body_color}</material>
+  <mu1>0.2</mu1>
+  <mu2>0.2</mu2>
+  <selfCollide>true</selfCollide>
+</gazebo>
+-->
 </robot>
