Commit message: ustbot low poly demo

File: src/Simulation/Descriptions/ustbot_description/urdf/ustbot.urdf.xacro (robot description, xacro)
@@ -1,18 +1,6 @@
-<?xml version="1.0" encoding="utf-8"?>
-<!-- This URDF was automatically created by SolidWorks to URDF Exporter! Originally created by Stephen Brawner (brawner@gmail.com)
-     Commit Version: 1.6.0-1-g15f4949  Build Version: 1.6.7594.29634
-     For more information, please see http://wiki.ros.org/sw_urdf_exporter -->
-<robot
-  name="ustbot"
-  xmlns:xacro="http://ros.org/wiki/xacro">
-  <xacro:include filename="$(find ustbot_description)/urdf/ustbot.gazebo.xacro"/>
-  <!-- Used for fixing robot to Gazebo 'base_link' -->
-  <!--
-  <link name="world"/>
-  <joint name="fixed" type="fixed">
-    <parent link="world"/>
-    <child link="link1"/>
-  </joint>
-  -->
+<?xml version="1.0" ?>
+<robot name="ustbot" xmlns:xacro="http://www.ros.org/wiki/xacro">
+<xacro:include filename="$(find ustbot_description)/urdf/materials.xacro" />
+<xacro:include filename="$(find ustbot_description)/urdf/ustbot.gazebo.xacro" />
   <link  name="base_footprint"/>
   <joint name="base_joint" type="fixed">
@@ -25,1505 +13,347 @@
       rpy="0 0 0"/>
   </joint>
-  <!-- ******************************************** -->
-  <!-- ********** Driven Wheels Section ********** -->
-  <link name="base_link">
-    <inertial>
-      <origin
-        xyz="0.013217 0.0075253 0.31131"
-        rpy="0 0 0" />
-      <mass
-        value="76.998" />
-      <inertia
-        ixx="1.9819"
-        ixy="0.0010984"
-        ixz="0.0010634"
-        iyy="1.9365"
-        iyz="-0.00042068"
-        izz="2.3951" />
-    </inertial>
-    <visual>
-      <origin
-        xyz="0 0 0"
-        rpy="0 0 0" />
-      <geometry>
-        <mesh
-          filename="package://ustbot_description/meshes/base_link.STL" />
-      </geometry>
-      <material
-        name="">
-        <color
-          rgba="0.89804 0.91765 0.92941 1" />
-      </material>
-    </visual>
-    <collision>
-      <origin
-        xyz="0 0 0"
-        rpy="0 0 0" />
-      <geometry>
-        <mesh
-          filename="package://ustbot_description/meshes/base_link.STL" />
-      </geometry>
-    </collision>
-  </link>
-  <link name="left_wheelhub_link">
-    <inertial>
-      <origin
-        xyz="2.1270092198097E-18 3.74115927137672E-06 0.0346504264024086"
-        rpy="0 0 0" />
-      <mass
-        value="3.07120221177258" />
-      <inertia
-        ixx="0.0054831110453997"
-        ixy="2.15571771255504E-22"
-        ixz="4.84300075074391E-19"
-        iyy="0.00548317428259655"
-        iyz="6.31372521057598E-07"
-        izz="0.00925980692151947" />
-    </inertial>
-    <visual>
-      <origin
-        xyz="0 0 0"
-        rpy="0 0 0" />
-      <geometry>
-        <mesh
-          filename="package://ustbot_description/meshes/left_wheelhub_link.STL" />
-      </geometry>
-      <material
-        name="">
-        <color
-          rgba="1 1 1 1" />
-      </material>
-    </visual>
-    <collision>
-      <origin
-        xyz="0 0 0"
-        rpy="0 0 0" />
-      <geometry>
-        <mesh
-          filename="package://ustbot_description/meshes/left_wheelhub_link.STL" />
-      </geometry>
-    </collision>
-  </link>
-  <joint name="left_wheelhub_joint" type="continuous">
-    <origin
-      xyz="0 0.19 0.005"
-      rpy="-1.5708 0 0" />
-    <parent
-      link="base_link" />
-    <child
-      link="left_wheelhub_link" />
-    <axis
-      xyz="0 0 1" />
-    <limit
-      lower="-10000"
-      upper="10000"
-      effort="1000"
-      velocity="1000" />
+<link name="base_link">
+  <inertial>
+    <origin xyz="-5.181182074625435e-16 0.0 0.155331106352338" rpy="0 0 0"/>
+    <mass value="54.59936129727744"/>
+    <inertia ixx="3.18013" iyy="4.05832" izz="6.857677" ixy="-2.7e-05" iyz="-0.0" ixz="-0.0"/>
+  </inertial>
+  <visual>
+    <origin xyz="0 0 0" rpy="0 0 0"/>
+    <geometry>
+      <mesh filename="package://ustbot_description/meshes2/base_link.stl" scale="0.001 0.001 0.001"/>
+    </geometry>
+    <material name="silver"/>
+  </visual>
+  <collision>
+    <origin xyz="0 0 0" rpy="0 0 0"/>
+    <geometry>
+      <mesh filename="package://ustbot_description/meshes2/base_link.stl" scale="0.001 0.001 0.001"/>
+    </geometry>
+  </collision>
+</link>
+<link name="wheel_right">
+  <inertial>
+    <origin xyz="1.215274427416404e-17 0.0 1.3877787807814457e-17" rpy="0 0 0"/>
+    <mass value="1.3919984714020586"/>
+    <inertia ixx="0.002937" iyy="0.004737" izz="0.002937" ixy="0.0" iyz="0.0" ixz="-0.0"/>
+  </inertial>
+  <visual>
+    <origin xyz="-0.0 0.225 -0.0825" rpy="0 0 0"/>
+    <geometry>
+      <mesh filename="package://ustbot_description/meshes2/wheel_right.stl" scale="0.001 0.001 0.001"/>
+    </geometry>
+    <material name="silver"/>
+  </visual>
+  <collision>
+    <origin xyz="-0.0 0.225 -0.0825" rpy="0 0 0"/>
+    <geometry>
+      <mesh filename="package://ustbot_description/meshes2/wheel_right.stl" scale="0.001 0.001 0.001"/>
+    </geometry>
+  </collision>
+</link>
+<link name="wheel_left">
+  <inertial>
+    <origin xyz="1.215274427416404e-17 0.0 1.3877787807814457e-17" rpy="0 0 0"/>
+    <mass value="1.3919984714020586"/>
+    <inertia ixx="0.002937" iyy="0.004737" izz="0.002937" ixy="-0.0" iyz="0.0" ixz="-0.0"/>
+  </inertial>
+  <visual>
+    <origin xyz="-0.0 -0.225 -0.0825" rpy="0 0 0"/>
+    <geometry>
+      <mesh filename="package://ustbot_description/meshes2/wheel_left.stl" scale="0.001 0.001 0.001"/>
+    </geometry>
+    <material name="silver"/>
+  </visual>
+  <collision>
+    <origin xyz="-0.0 -0.225 -0.0825" rpy="0 0 0"/>
+    <geometry>
+      <mesh filename="package://ustbot_description/meshes2/wheel_left.stl" scale="0.001 0.001 0.001"/>
+    </geometry>
+  </collision>
+</link>
+<link name="ultrasonic_front_right">
+  <inertial>
+    <origin xyz="0.0025000000000000577 -1.3013724642352287e-07 0.0" rpy="0 0 0"/>
+    <mass value="0.04471200116533985"/>
+    <inertia ixx="1e-05" iyy="2e-06" izz="8e-06" ixy="0.0" iyz="-0.0" ixz="-0.0"/>
+  </inertial>
+  <visual>
+    <origin xyz="-0.44501 0.172077 -0.1955" rpy="0 0 0"/>
+    <geometry>
+      <mesh filename="package://ustbot_description/meshes2/ultrasonic_front_right.stl" scale="0.001 0.001 0.001"/>
+    </geometry>
+    <material name="silver"/>
+  </visual>
+  <collision>
+    <origin xyz="-0.44501 0.172077 -0.1955" rpy="0 0 0"/>
+    <geometry>
+      <mesh filename="package://ustbot_description/meshes2/ultrasonic_front_right.stl" scale="0.001 0.001 0.001"/>
+    </geometry>
+  </collision>
+</link>
+<link name="ultrasonic_front_left">
+  <inertial>
+    <origin xyz="0.0025000000000000577 1.3013724642352287e-07 0.0" rpy="0 0 0"/>
+    <mass value="0.04471200116533985"/>
+    <inertia ixx="1e-05" iyy="2e-06" izz="8e-06" ixy="-0.0" iyz="0.0" ixz="-0.0"/>
+  </inertial>
+  <visual>
+    <origin xyz="-0.44501 -0.172077 -0.1955" rpy="0 0 0"/>
+    <geometry>
+      <mesh filename="package://ustbot_description/meshes2/ultrasonic_front_left.stl" scale="0.001 0.001 0.001"/>
+    </geometry>
+    <material name="silver"/>
+  </visual>
+  <collision>
+    <origin xyz="-0.44501 -0.172077 -0.1955" rpy="0 0 0"/>
+    <geometry>
+      <mesh filename="package://ustbot_description/meshes2/ultrasonic_front_left.stl" scale="0.001 0.001 0.001"/>
+    </geometry>
+  </collision>
+</link>
+<link name="ultrasonic_left_left">
+  <inertial>
+    <origin xyz="-1.88564546477199e-07 0.0025000000000000577 0.0" rpy="0 0 0"/>
+    <mass value="0.04471200116533985"/>
+    <inertia ixx="2e-06" iyy="1e-05" izz="8e-06" ixy="0.0" iyz="-0.0" ixz="0.0"/>
+  </inertial>
+  <visual>
+    <origin xyz="-0.313812 -0.30001 -0.1955" rpy="0 0 0"/>
+    <geometry>
+      <mesh filename="package://ustbot_description/meshes2/ultrasonic_left_left.stl" scale="0.001 0.001 0.001"/>
+    </geometry>
+    <material name="silver"/>
+  </visual>
+  <collision>
+    <origin xyz="-0.313812 -0.30001 -0.1955" rpy="0 0 0"/>
+    <geometry>
+      <mesh filename="package://ustbot_description/meshes2/ultrasonic_left_left.stl" scale="0.001 0.001 0.001"/>
+    </geometry>
+  </collision>
+</link>
+<link name="ultrasonic_left_right">
+  <inertial>
+    <origin xyz="1.88564546477199e-07 0.0025000000000000577 0.0" rpy="0 0 0"/>
+    <mass value="0.04471200116533985"/>
+    <inertia ixx="2e-06" iyy="1e-05" izz="8e-06" ixy="-0.0" iyz="-0.0" ixz="-0.0"/>
+  </inertial>
+  <visual>
+    <origin xyz="0.313812 -0.30001 -0.1955" rpy="0 0 0"/>
+    <geometry>
+      <mesh filename="package://ustbot_description/meshes2/ultrasonic_left_right.stl" scale="0.001 0.001 0.001"/>
+    </geometry>
+    <material name="silver"/>
+  </visual>
+  <collision>
+    <origin xyz="0.313812 -0.30001 -0.1955" rpy="0 0 0"/>
+    <geometry>
+      <mesh filename="package://ustbot_description/meshes2/ultrasonic_left_right.stl" scale="0.001 0.001 0.001"/>
+    </geometry>
+  </collision>
+</link>
+<link name="ultrasonic_back_left">
+  <inertial>
+    <origin xyz="-0.0025000000000000577 1.3013724642352287e-07 0.0" rpy="0 0 0"/>
+    <mass value="0.044712001165339924"/>
+    <inertia ixx="1e-05" iyy="2e-06" izz="8e-06" ixy="0.0" iyz="0.0" ixz="0.0"/>
+  </inertial>
+  <visual>
+    <origin xyz="0.44501 -0.172077 -0.1955" rpy="0 0 0"/>
+    <geometry>
+      <mesh filename="package://ustbot_description/meshes2/ultrasonic_back_left.stl" scale="0.001 0.001 0.001"/>
+    </geometry>
+    <material name="silver"/>
+  </visual>
+  <collision>
+    <origin xyz="0.44501 -0.172077 -0.1955" rpy="0 0 0"/>
+    <geometry>
+      <mesh filename="package://ustbot_description/meshes2/ultrasonic_back_left.stl" scale="0.001 0.001 0.001"/>
+    </geometry>
+  </collision>
+</link>
+<link name="ultrasonic_back_right">
+  <inertial>
+    <origin xyz="-0.0025000000000000577 -1.3013724642352287e-07 0.0" rpy="0 0 0"/>
+    <mass value="0.044712001165339924"/>
+    <inertia ixx="1e-05" iyy="2e-06" izz="8e-06" ixy="-0.0" iyz="-0.0" ixz="0.0"/>
+  </inertial>
+  <visual>
+    <origin xyz="0.44501 0.172077 -0.1955" rpy="0 0 0"/>
+    <geometry>
+      <mesh filename="package://ustbot_description/meshes2/ultrasonic_back_right.stl" scale="0.001 0.001 0.001"/>
+    </geometry>
+    <material name="silver"/>
+  </visual>
+  <collision>
+    <origin xyz="0.44501 0.172077 -0.1955" rpy="0 0 0"/>
+    <geometry>
+      <mesh filename="package://ustbot_description/meshes2/ultrasonic_back_right.stl" scale="0.001 0.001 0.001"/>
+    </geometry>
+  </collision>
+</link>
+<link name="ultrasonic_right_left">
+  <inertial>
+    <origin xyz="1.88564546477199e-07 -0.0025000000000000577 0.0" rpy="0 0 0"/>
+    <mass value="0.04471200116533992"/>
+    <inertia ixx="2e-06" iyy="1e-05" izz="8e-06" ixy="-0.0" iyz="0.0" ixz="0.0"/>
+  </inertial>
+  <visual>
+    <origin xyz="0.313812 0.30001 -0.1955" rpy="0 0 0"/>
+    <geometry>
+      <mesh filename="package://ustbot_description/meshes2/ultrasonic_right_left.stl" scale="0.001 0.001 0.001"/>
+    </geometry>
+    <material name="silver"/>
+  </visual>
+  <collision>
+    <origin xyz="0.313812 0.30001 -0.1955" rpy="0 0 0"/>
+    <geometry>
+      <mesh filename="package://ustbot_description/meshes2/ultrasonic_right_left.stl" scale="0.001 0.001 0.001"/>
+    </geometry>
+  </collision>
+</link>
+<link name="ultrasonic_right_right">
+  <inertial>
+    <origin xyz="-1.8856454653271015e-07 -0.0025000000000000577 0.0" rpy="0 0 0"/>
+    <mass value="0.04471200116533992"/>
+    <inertia ixx="2e-06" iyy="1e-05" izz="8e-06" ixy="0.0" iyz="0.0" ixz="-0.0"/>
+  </inertial>
+  <visual>
+    <origin xyz="-0.313812 0.30001 -0.1955" rpy="0 0 0"/>
+    <geometry>
+      <mesh filename="package://ustbot_description/meshes2/ultrasonic_right_right.stl" scale="0.001 0.001 0.001"/>
+    </geometry>
+    <material name="silver"/>
+  </visual>
+  <collision>
+    <origin xyz="-0.313812 0.30001 -0.1955" rpy="0 0 0"/>
+    <geometry>
+      <mesh filename="package://ustbot_description/meshes2/ultrasonic_right_right.stl" scale="0.001 0.001 0.001"/>
+    </geometry>
+  </collision>
+</link>
+<link name="lidar_front">
+  <inertial>
+    <origin xyz="-5.551115123125783e-17 5.551115123125783e-17 0.017500000000000016" rpy="0 0 0"/>
+    <mass value="0.1356625159140251"/>
+    <inertia ixx="5.8e-05" iyy="5.8e-05" izz="8.8e-05" ixy="0.0" iyz="0.0" ixz="0.0"/>
+  </inertial>
+  <visual>
+    <origin xyz="-0.386 -0.241 -0.23751" rpy="0 0 0"/>
+    <geometry>
+      <mesh filename="package://ustbot_description/meshes2/lidar_front.stl" scale="0.001 0.001 0.001"/>
+    </geometry>
+    <material name="silver"/>
+  </visual>
+  <collision>
+    <origin xyz="-0.386 -0.241 -0.23751" rpy="0 0 0"/>
+    <geometry>
+      <mesh filename="package://ustbot_description/meshes2/lidar_front.stl" scale="0.001 0.001 0.001"/>
+    </geometry>
+  </collision>
+</link>
+<link name="lidar_back">
+  <inertial>
+    <origin xyz="0.0 0.0 0.01749999999999996" rpy="0 0 0"/>
+    <mass value="0.1356625159140251"/>
+    <inertia ixx="5.8e-05" iyy="5.8e-05" izz="8.8e-05" ixy="0.0" iyz="0.0" ixz="-0.0"/>
+  </inertial>
+  <visual>
+    <origin xyz="0.386 0.241 -0.23751" rpy="0 0 0"/>
+    <geometry>
+      <mesh filename="package://ustbot_description/meshes2/lidar_back.stl" scale="0.001 0.001 0.001"/>
+    </geometry>
+    <material name="silver"/>
+  </visual>
+  <collision>
+    <origin xyz="0.386 0.241 -0.23751" rpy="0 0 0"/>
+    <geometry>
+      <mesh filename="package://ustbot_description/meshes2/lidar_back.stl" scale="0.001 0.001 0.001"/>
+    </geometry>
+  </collision>
+</link>
+<joint name="wheel_right_joint" type="continuous">
+  <origin xyz="0.0 -0.225 0.0825" rpy="0 0 0"/>
+  <parent link="base_link"/>
+  <child link="wheel_right"/>
+  <axis xyz="0.0 1.0 0.0"/>
+</joint>
+<joint name="wheel_left_joint" type="continuous">
+  <origin xyz="0.0 0.225 0.0825" rpy="0 0 0"/>
+  <parent link="base_link"/>
+  <child link="wheel_left"/>
+  <axis xyz="0.0 1.0 0.0"/>
+</joint>
+<joint name="ultrasonic_front_right" type="fixed">
+  <origin xyz="0.44501 -0.172077 0.1955" rpy="0 0 0"/>
+  <parent link="base_link"/>
+  <child link="ultrasonic_front_right"/>
+</joint>
+<joint name="ultrasonic_front_left" type="fixed">
+  <origin xyz="0.44501 0.172077 0.1955" rpy="0 0 0"/>
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