Commit message: Removing controller spawner since we are going to use the libgazebo_ros_diff_drive

File: src/Simulation/Descriptions/ustbot_description/urdf/ustbot.gazebo.xacro (robot description, xacro)
@@ -2,10 +2,4 @@
 <robot name="ustbot" xmlns:xacro="http://www.ros.org/wiki/xacro" >
 <xacro:property name="body_color" value="Gazebo/Silver" />
-<!--
-<gazebo>
-  <plugin name="gazebo_ros_control" filename="libgazebo_ros_control.so">
-  </plugin>
-</gazebo>
--->
 <gazebo>
   <plugin name="ustbot_controller" filename="libgazebo_ros_diff_drive.so">
@@ -26,17 +20,16 @@
     <wheelDiameter>0.165</wheelDiameter>
     <wheelAcceleration>1</wheelAcceleration>
-    <wheelTorque>100</wheelTorque>
+    <wheelTorque>70</wheelTorque>
     <rosDebugLevel>na</rosDebugLevel>
   </plugin>
 </gazebo>
 <gazebo reference="base_link">
-  <material>${body_color}</material>
-  <mu1>0.1</mu1>
-  <mu2>0.1</mu2>
-  <selfCollide>true</selfCollide>
+  <material>Gazebo/DarkGrey </material>
+  <mu1>0.05</mu1>
+  <mu2>0.05</mu2>
   <gravity>true</gravity>
 </gazebo>
 <gazebo reference="wheel_right">
-  <material>${body_color}</material>
+  <material>Gazebo/FlatBlack</material>
   <mu1>3500</mu1>
   <mu2>3500</mu2>
@@ -44,7 +37,15 @@
 </gazebo>
 <gazebo reference="wheel_left">
-  <material>${body_color}</material>
+  <material>Gazebo/FlatBlack</material>
   <mu1>3500</mu1>
   <mu2>3500</mu2>
+  <selfCollide>true</selfCollide>
+</gazebo>
+<gazebo reference="lidar_front">
+  <material>Gazebo/Blue</material>
+  <selfCollide>true</selfCollide>
+</gazebo>
+<gazebo reference="lidar_back">
+  <material>Gazebo/Blue</material>
   <selfCollide>true</selfCollide>
 </gazebo>
@@ -98,16 +99,4 @@
   <selfCollide>true</selfCollide>
 </gazebo>
-<gazebo reference="lidar_front">
-  <material>${body_color}</material>
-  <mu1>0.2</mu1>
-  <mu2>0.2</mu2>
-  <selfCollide>true</selfCollide>
-</gazebo>
-<gazebo reference="lidar_back">
-  <material>${body_color}</material>
-  <mu1>0.2</mu1>
-  <mu2>0.2</mu2>
-  <selfCollide>true</selfCollide>
-</gazebo>
 -->
 </robot>

File: src/Simulation/Descriptions/ustbot_description/urdf/ustbot.urdf.xacro (robot description, xacro)
@@ -22,12 +22,11 @@
     <origin xyz="0 0 0" rpy="0 0 0"/>
     <geometry>
-      <mesh filename="package://ustbot_description/meshes2/base_link.stl" scale="0.001 0.001 0.001"/>
-    </geometry>
-    <material name="silver"/>
+      <mesh filename="package://ustbot_description/meshes/base_link.STL" scale="0.001 0.001 0.001"/>
+    </geometry>
   </visual>
   <collision>
     <origin xyz="0 0 0" rpy="0 0 0"/>
     <geometry>
-      <mesh filename="package://ustbot_description/meshes2/base_link.stl" scale="0.001 0.001 0.001"/>
+      <mesh filename="package://ustbot_description/meshes/base_link.STL" scale="0.001 0.001 0.001"/>
     </geometry>
   </collision>
@@ -42,12 +41,11 @@
     <origin xyz="-0.0 0.225 -0.0825" rpy="0 0 0"/>
     <geometry>
-      <mesh filename="package://ustbot_description/meshes2/wheel_right.stl" scale="0.001 0.001 0.001"/>
-    </geometry>
-    <material name="silver"/>
+      <mesh filename="package://ustbot_description/meshes/wheel_right.STL" scale="0.001 0.001 0.001"/>
+    </geometry>
   </visual>
   <collision>
     <origin xyz="-0.0 0.225 -0.0825" rpy="0 0 0"/>
     <geometry>
-      <mesh filename="package://ustbot_description/meshes2/wheel_right.stl" scale="0.001 0.001 0.001"/>
+      <mesh filename="package://ustbot_description/meshes/wheel_right.STL" scale="0.001 0.001 0.001"/>
     </geometry>
   </collision>
@@ -62,12 +60,11 @@
     <origin xyz="-0.0 -0.225 -0.0825" rpy="0 0 0"/>
     <geometry>
-      <mesh filename="package://ustbot_description/meshes2/wheel_left.stl" scale="0.001 0.001 0.001"/>
-    </geometry>
-    <material name="silver"/>
+      <mesh filename="package://ustbot_description/meshes/wheel_left.STL" scale="0.001 0.001 0.001"/>
+    </geometry>
   </visual>
   <collision>
     <origin xyz="-0.0 -0.225 -0.0825" rpy="0 0 0"/>
     <geometry>
-      <mesh filename="package://ustbot_description/meshes2/wheel_left.stl" scale="0.001 0.001 0.001"/>
+      <mesh filename="package://ustbot_description/meshes/wheel_left.STL" scale="0.001 0.001 0.001"/>
     </geometry>
   </collision>
@@ -82,12 +79,11 @@
     <origin xyz="-0.44501 0.172077 -0.1955" rpy="0 0 0"/>
     <geometry>
-      <mesh filename="package://ustbot_description/meshes2/ultrasonic_front_right.stl" scale="0.001 0.001 0.001"/>
-    </geometry>
-    <material name="silver"/>
+      <mesh filename="package://ustbot_description/meshes/ultrasonic_front_right.STL" scale="0.001 0.001 0.001"/>
+    </geometry>
   </visual>
   <collision>
     <origin xyz="-0.44501 0.172077 -0.1955" rpy="0 0 0"/>
     <geometry>
-      <mesh filename="package://ustbot_description/meshes2/ultrasonic_front_right.stl" scale="0.001 0.001 0.001"/>
+      <mesh filename="package://ustbot_description/meshes/ultrasonic_front_right.STL" scale="0.001 0.001 0.001"/>
     </geometry>
   </collision>
@@ -102,12 +98,11 @@
     <origin xyz="-0.44501 -0.172077 -0.1955" rpy="0 0 0"/>
     <geometry>
-      <mesh filename="package://ustbot_description/meshes2/ultrasonic_front_left.stl" scale="0.001 0.001 0.001"/>
-    </geometry>
-    <material name="silver"/>
+      <mesh filename="package://ustbot_description/meshes/ultrasonic_front_left.STL" scale="0.001 0.001 0.001"/>
+    </geometry>
   </visual>
   <collision>
     <origin xyz="-0.44501 -0.172077 -0.1955" rpy="0 0 0"/>
     <geometry>
-      <mesh filename="package://ustbot_description/meshes2/ultrasonic_front_left.stl" scale="0.001 0.001 0.001"/>
+      <mesh filename="package://ustbot_description/meshes/ultrasonic_front_left.STL" scale="0.001 0.001 0.001"/>
     </geometry>
   </collision>
@@ -122,12 +117,11 @@
     <origin xyz="-0.313812 -0.30001 -0.1955" rpy="0 0 0"/>
     <geometry>
-      <mesh filename="package://ustbot_description/meshes2/ultrasonic_left_left.stl" scale="0.001 0.001 0.001"/>
-    </geometry>
-    <material name="silver"/>
+      <mesh filename="package://ustbot_description/meshes/ultrasonic_left_left.STL" scale="0.001 0.001 0.001"/>
+    </geometry>
   </visual>
   <collision>
     <origin xyz="-0.313812 -0.30001 -0.1955" rpy="0 0 0"/>
     <geometry>
-      <mesh filename="package://ustbot_description/meshes2/ultrasonic_left_left.stl" scale="0.001 0.001 0.001"/>
+      <mesh filename="package://ustbot_description/meshes/ultrasonic_left_left.STL" scale="0.001 0.001 0.001"/>
     </geometry>
   </collision>
@@ -142,12 +136,11 @@
     <origin xyz="0.313812 -0.30001 -0.1955" rpy="0 0 0"/>
     <geometry>
-      <mesh filename="package://ustbot_description/meshes2/ultrasonic_left_right.stl" scale="0.001 0.001 0.001"/>
-    </geometry>
-    <material name="silver"/>
+      <mesh filename="package://ustbot_description/meshes/ultrasonic_left_right.STL" scale="0.001 0.001 0.001"/>
+    </geometry>
   </visual>
   <collision>
     <origin xyz="0.313812 -0.30001 -0.1955" rpy="0 0 0"/>
     <geometry>
-      <mesh filename="package://ustbot_description/meshes2/ultrasonic_left_right.stl" scale="0.001 0.001 0.001"/>
+      <mesh filename="package://ustbot_description/meshes/ultrasonic_left_right.STL" scale="0.001 0.001 0.001"/>
     </geometry>
   </collision>
@@ -162,12 +155,11 @@
     <origin xyz="0.44501 -0.172077 -0.1955" rpy="0 0 0"/>
     <geometry>
-      <mesh filename="package://ustbot_description/meshes2/ultrasonic_back_left.stl" scale="0.001 0.001 0.001"/>
-    </geometry>
-    <material name="silver"/>
+      <mesh filename="package://ustbot_description/meshes/ultrasonic_back_left.STL" scale="0.001 0.001 0.001"/>
+    </geometry>
   </visual>
   <collision>
     <origin xyz="0.44501 -0.172077 -0.1955" rpy="0 0 0"/>
     <geometry>
-      <mesh filename="package://ustbot_description/meshes2/ultrasonic_back_left.stl" scale="0.001 0.001 0.001"/>
+      <mesh filename="package://ustbot_description/meshes/ultrasonic_back_left.STL" scale="0.001 0.001 0.001"/>
     </geometry>
   </collision>
@@ -182,12 +174,11 @@
     <origin xyz="0.44501 0.172077 -0.1955" rpy="0 0 0"/>
     <geometry>
-      <mesh filename="package://ustbot_description/meshes2/ultrasonic_back_right.stl" scale="0.001 0.001 0.001"/>
-    </geometry>
-    <material name="silver"/>
+      <mesh filename="package://ustbot_description/meshes/ultrasonic_back_right.STL" scale="0.001 0.001 0.001"/>
+    </geometry>
   </visual>
   <collision>
     <origin xyz="0.44501 0.172077 -0.1955" rpy="0 0 0"/>
     <geometry>
-      <mesh filename="package://ustbot_description/meshes2/ultrasonic_back_right.stl" scale="0.001 0.001 0.001"/>
+      <mesh filename="package://ustbot_description/meshes/ultrasonic_back_right.STL" scale="0.001 0.001 0.001"/>
     </geometry>
   </collision>
@@ -202,12 +193,11 @@
     <origin xyz="0.313812 0.30001 -0.1955" rpy="0 0 0"/>
     <geometry>
-      <mesh filename="package://ustbot_description/meshes2/ultrasonic_right_left.stl" scale="0.001 0.001 0.001"/>
-    </geometry>
-    <material name="silver"/>
+      <mesh filename="package://ustbot_description/meshes/ultrasonic_right_left.STL" scale="0.001 0.001 0.001"/>
+    </geometry>
   </visual>
   <collision>
     <origin xyz="0.313812 0.30001 -0.1955" rpy="0 0 0"/>
     <geometry>
-      <mesh filename="package://ustbot_description/meshes2/ultrasonic_right_left.stl" scale="0.001 0.001 0.001"/>
+      <mesh filename="package://ustbot_description/meshes/ultrasonic_right_left.STL" scale="0.001 0.001 0.001"/>
     </geometry>
   </collision>
@@ -222,12 +212,11 @@
     <origin xyz="-0.313812 0.30001 -0.1955" rpy="0 0 0"/>
     <geometry>
-      <mesh filename="package://ustbot_description/meshes2/ultrasonic_right_right.stl" scale="0.001 0.001 0.001"/>
-    </geometry>
-    <material name="silver"/>
+      <mesh filename="package://ustbot_description/meshes/ultrasonic_right_right.STL" scale="0.001 0.001 0.001"/>
+    </geometry>
   </visual>
   <collision>
     <origin xyz="-0.313812 0.30001 -0.1955" rpy="0 0 0"/>
     <geometry>
-      <mesh filename="package://ustbot_description/meshes2/ultrasonic_right_right.stl" scale="0.001 0.001 0.001"/>
+      <mesh filename="package://ustbot_description/meshes/ultrasonic_right_right.STL" scale="0.001 0.001 0.001"/>
     </geometry>
   </collision>
@@ -242,12 +231,11 @@
     <origin xyz="-0.386 -0.241 -0.23751" rpy="0 0 0"/>
     <geometry>
-      <mesh filename="package://ustbot_description/meshes2/lidar_front.stl" scale="0.001 0.001 0.001"/>
-    </geometry>
-    <material name="silver"/>
+      <mesh filename="package://ustbot_description/meshes/lidar_front.STL" scale="0.001 0.001 0.001"/>
+    </geometry>
   </visual>
   <collision>
     <origin xyz="-0.386 -0.241 -0.23751" rpy="0 0 0"/>
     <geometry>
-      <mesh filename="package://ustbot_description/meshes2/lidar_front.stl" scale="0.001 0.001 0.001"/>
+      <mesh filename="package://ustbot_description/meshes/lidar_front.STL" scale="0.001 0.001 0.001"/>
     </geometry>
   </collision>
@@ -262,12 +250,11 @@
     <origin xyz="0.386 0.241 -0.23751" rpy="0 0 0"/>
     <geometry>
-      <mesh filename="package://ustbot_description/meshes2/lidar_back.stl" scale="0.001 0.001 0.001"/>
-    </geometry>
-    <material name="silver"/>
+      <mesh filename="package://ustbot_description/meshes/lidar_back.STL" scale="0.001 0.001 0.001"/>
+    </geometry>
   </visual>
   <collision>
     <origin xyz="0.386 0.241 -0.23751" rpy="0 0 0"/>
     <geometry>
-      <mesh filename="package://ustbot_description/meshes2/lidar_back.stl" scale="0.001 0.001 0.001"/>
+      <mesh filename="package://ustbot_description/meshes/lidar_back.STL" scale="0.001 0.001 0.001"/>
     </geometry>
   </collision>

Commit message: Implementing lidars in simulation and including merging laser data package for merging laser data streams into one topic

File: src/Simulation/Descriptions/ustbot_description/urdf/ustbot.gazebo.xacro (robot description, xacro)
@@ -1,102 +1,169 @@
 <?xml version="1.0" ?>
 <robot name="ustbot" xmlns:xacro="http://www.ros.org/wiki/xacro" >
-<xacro:property name="body_color" value="Gazebo/Silver" />
-<gazebo>
-  <plugin name="ustbot_controller" filename="libgazebo_ros_diff_drive.so">
-    <commandTopic>cmd_vel</commandTopic>
-    <odometryTopic>odom</odometryTopic>
-    <odometryFrame>odom</odometryFrame>
-    <odometrySource>world</odometrySource>
-    <publishOdomTF>true</publishOdomTF>
-    <robotBaseFrame>base_footprint</robotBaseFrame>
-    <publishWheelTF>false</publishWheelTF>
-    <publishTf>true</publishTf>
-    <publishWheelJointState>true</publishWheelJointState>
-    <legacyMode>false</legacyMode>
-    <updateRate>30</updateRate>
-    <leftJoint>wheel_left_joint</leftJoint>
-    <rightJoint>wheel_right_joint</rightJoint>
-    <wheelSeparation>0.45</wheelSeparation>
-    <wheelDiameter>0.165</wheelDiameter>
-    <wheelAcceleration>1</wheelAcceleration>
-    <wheelTorque>70</wheelTorque>
-    <rosDebugLevel>na</rosDebugLevel>
-  </plugin>
-</gazebo>
-<gazebo reference="base_link">
-  <material>Gazebo/DarkGrey </material>
-  <mu1>0.05</mu1>
-  <mu2>0.05</mu2>
-  <gravity>true</gravity>
-</gazebo>
-<gazebo reference="wheel_right">
-  <material>Gazebo/FlatBlack</material>
-  <mu1>3500</mu1>
-  <mu2>3500</mu2>
-  <selfCollide>true</selfCollide>
-</gazebo>
-<gazebo reference="wheel_left">
-  <material>Gazebo/FlatBlack</material>
-  <mu1>3500</mu1>
-  <mu2>3500</mu2>
-  <selfCollide>true</selfCollide>
-</gazebo>
-<gazebo reference="lidar_front">
-  <material>Gazebo/Blue</material>
-  <selfCollide>true</selfCollide>
-</gazebo>
-<gazebo reference="lidar_back">
-  <material>Gazebo/Blue</material>
-  <selfCollide>true</selfCollide>
-</gazebo>
-<!--
-<gazebo reference="ultrasonic_front_right">
-  <material>${body_color}</material>
-  <mu1>0.2</mu1>
-  <mu2>0.2</mu2>
-  <selfCollide>true</selfCollide>
-</gazebo>
-<gazebo reference="ultrasonic_front_left">
-  <material>${body_color}</material>
-  <mu1>0.2</mu1>
-  <mu2>0.2</mu2>
-  <selfCollide>true</selfCollide>
-</gazebo>
-<gazebo reference="ultrasonic_left_left">
-  <material>${body_color}</material>
-  <mu1>0.2</mu1>
-  <mu2>0.2</mu2>
-  <selfCollide>true</selfCollide>
-</gazebo>
-<gazebo reference="ultrasonic_left_right">
-  <material>${body_color}</material>
-  <mu1>0.2</mu1>
-  <mu2>0.2</mu2>
-  <selfCollide>true</selfCollide>
-</gazebo>
-<gazebo reference="ultrasonic_back_left">
-  <material>${body_color}</material>
-  <mu1>0.2</mu1>
-  <mu2>0.2</mu2>
-  <selfCollide>true</selfCollide>
-</gazebo>
-<gazebo reference="ultrasonic_back_right">
-  <material>${body_color}</material>
-  <mu1>0.2</mu1>
-  <mu2>0.2</mu2>
-  <selfCollide>true</selfCollide>
-</gazebo>
-<gazebo reference="ultrasonic_right_left">
-  <material>${body_color}</material>
-  <mu1>0.2</mu1>
-  <mu2>0.2</mu2>
-  <selfCollide>true</selfCollide>
-</gazebo>
-<gazebo reference="ultrasonic_right_right">
-  <material>${body_color}</material>
-  <mu1>0.2</mu1>
-  <mu2>0.2</mu2>
-  <selfCollide>true</selfCollide>
-</gazebo>
--->
+  <xacro:arg name="laser_visual" default="false"/>
+  <xacro:property name="body_color" value="Gazebo/Silver" />
+  <gazebo>
+    <plugin name="ustbot_controller" filename="libgazebo_ros_diff_drive.so">
+      <commandTopic>cmd_vel</commandTopic>
+      <odometryTopic>odom</odometryTopic>
+      <odometryFrame>odom</odometryFrame>
+      <odometrySource>world</odometrySource>
+      <publishOdomTF>true</publishOdomTF>
+      <robotBaseFrame>base_footprint</robotBaseFrame>
+      <publishWheelTF>false</publishWheelTF>
+      <publishTf>true</publishTf>
+      <publishWheelJointState>true</publishWheelJointState>
+      <legacyMode>false</legacyMode>
+      <updateRate>30</updateRate>
+      <leftJoint>wheel_left_joint</leftJoint>
+      <rightJoint>wheel_right_joint</rightJoint>
+      <wheelSeparation>0.45</wheelSeparation>
+      <wheelDiameter>0.165</wheelDiameter>
+      <wheelAcceleration>1</wheelAcceleration>
+      <wheelTorque>70</wheelTorque>
+      <rosDebugLevel>na</rosDebugLevel>
+    </plugin>
+  </gazebo>
+  <!-- *********** simulated ray sensor FRONT side *********** -->
+  <gazebo reference="lidar_front">
+    <material>Gazebo/FlatBlack</material>
+    <sensor type="ray" name="lidar_front_sensor">
+      <pose>0 0 0 0 0 0</pose>
+      <visualize>$(arg laser_visual)</visualize>
+      <update_rate>5</update_rate>
+      <ray>
+        <scan>
+          <horizontal>
+            <samples>360</samples>
+            <resolution>1</resolution>
+            <min_angle>-1.5708</min_angle>
+            <max_angle>3.1416</max_angle>
+          </horizontal>
+        </scan>
+        <range>
+          <min>0.120</min>
+          <max>3.5</max>
+          <resolution>0.015</resolution>
+        </range>
+        <noise>
+          <type>gaussian</type>
+          <mean>0.0</mean>
+          <stddev>0.01</stddev>
+        </noise>
+      </ray>
+      <plugin name="gazebo_ros_lidar_front_controller" filename="libgazebo_ros_laser.so">
+        <topicName>scan_front</topicName>
+        <frameName>lidar_front</frameName>
+      </plugin>
+    </sensor>
+  </gazebo>
+  <!-- *********** simulated ray sensor BACK side *********** -->
+  <gazebo reference="lidar_back">
+    <material>Gazebo/FlatBlack</material>
+    <sensor type="ray" name="lidar_back_sensor">
+      <pose>0 0 0 0 0 0</pose>
+      <visualize>$(arg laser_visual)</visualize>
+      <update_rate>5</update_rate>
+      <ray>
+        <scan>
+          <horizontal>
+            <samples>360</samples>
+            <resolution>1</resolution>
+            <min_angle>1.5708</min_angle>
+            <max_angle>6.28319</max_angle>
+          </horizontal>
+        </scan>
+        <range>
+          <min>0.120</min>
+          <max>3.5</max>
+          <resolution>0.015</resolution>
+        </range>
+        <noise>
+          <type>gaussian</type>
+          <mean>0.0</mean>
+          <stddev>0.01</stddev>
+        </noise>
+      </ray>
+      <plugin name="gazebo_ros_lidar_back_controller" filename="libgazebo_ros_laser.so">
+        <topicName>scan_back</topicName>
+        <frameName>lidar_back</frameName>
+      </plugin>
+    </sensor>
+  </gazebo>
+  <gazebo reference="base_link">
+    <material>Gazebo/DarkGrey </material>
+    <mu1>0.05</mu1>
+    <mu2>0.05</mu2>
+    <gravity>true</gravity>
+  </gazebo>
+  <gazebo reference="wheel_right">
+    <material>Gazebo/FlatBlack</material>
+    <mu1>3500</mu1>
+    <mu2>3500</mu2>
+    <selfCollide>true</selfCollide>
+  </gazebo>
+  <gazebo reference="wheel_left">
+    <material>Gazebo/FlatBlack</material>
+    <mu1>3500</mu1>
+    <mu2>3500</mu2>
+    <selfCollide>true</selfCollide>
+  </gazebo>
+  <gazebo reference="lidar_front">
+    <material>Gazebo/Blue</material>
+    <selfCollide>true</selfCollide>
+  </gazebo>
+  <gazebo reference="lidar_back">
+    <material>Gazebo/Blue</material>
+    <selfCollide>true</selfCollide>
+  </gazebo>
+  <!--
+  <gazebo reference="ultrasonic_front_right">
+    <material>${body_color}</material>
+    <mu1>0.2</mu1>
+    <mu2>0.2</mu2>
+    <selfCollide>true</selfCollide>
+  </gazebo>
+  <gazebo reference="ultrasonic_front_left">
+    <material>${body_color}</material>
+    <mu1>0.2</mu1>
+    <mu2>0.2</mu2>
+    <selfCollide>true</selfCollide>
+  </gazebo>
+  <gazebo reference="ultrasonic_left_left">
+    <material>${body_color}</material>
+    <mu1>0.2</mu1>
+    <mu2>0.2</mu2>
+    <selfCollide>true</selfCollide>
+  </gazebo>
+  <gazebo reference="ultrasonic_left_right">
+    <material>${body_color}</material>
+    <mu1>0.2</mu1>
+    <mu2>0.2</mu2>
+    <selfCollide>true</selfCollide>
+  </gazebo>
+  <gazebo reference="ultrasonic_back_left">
+    <material>${body_color}</material>
+    <mu1>0.2</mu1>
+    <mu2>0.2</mu2>
+    <selfCollide>true</selfCollide>
+  </gazebo>
+  <gazebo reference="ultrasonic_back_right">
+    <material>${body_color}</material>
+    <mu1>0.2</mu1>
+    <mu2>0.2</mu2>
+    <selfCollide>true</selfCollide>
+  </gazebo>
+  <gazebo reference="ultrasonic_right_left">
+    <material>${body_color}</material>
+    <mu1>0.2</mu1>
+    <mu2>0.2</mu2>
+    <selfCollide>true</selfCollide>
+  </gazebo>
+  <gazebo reference="ultrasonic_right_right">
+    <material>${body_color}</material>
+    <mu1>0.2</mu1>
+    <mu2>0.2</mu2>
+    <selfCollide>true</selfCollide>
+  </gazebo>
+  -->
 </robot>

File: src/Simulation/Descriptions/ustbot_description/urdf/ustbot.urdf.xacro (robot description, xacro)
@@ -229,5 +229,5 @@
   </inertial>
   <visual>
-    <origin xyz="-0.386 -0.241 -0.23751" rpy="0 0 0"/>
+    <origin xyz="-0.386 -0.241 -0.25751" rpy="0 0 0"/>
     <geometry>
       <mesh filename="package://ustbot_description/meshes/lidar_front.STL" scale="0.001 0.001 0.001"/>
@@ -235,5 +235,5 @@
   </visual>
   <collision>
-    <origin xyz="-0.386 -0.241 -0.23751" rpy="0 0 0"/>
+    <origin xyz="-0.386 -0.241 -0.25751" rpy="0 0 0"/>
     <geometry>
       <mesh filename="package://ustbot_description/meshes/lidar_front.STL" scale="0.001 0.001 0.001"/>
@@ -248,5 +248,5 @@
   </inertial>
   <visual>
-    <origin xyz="0.386 0.241 -0.23751" rpy="0 0 0"/>
+    <origin xyz="0.386 0.241 -0.25751" rpy="0 0 0"/>
     <geometry>
       <mesh filename="package://ustbot_description/meshes/lidar_back.STL" scale="0.001 0.001 0.001"/>
@@ -254,5 +254,5 @@
   </visual>
   <collision>
-    <origin xyz="0.386 0.241 -0.23751" rpy="0 0 0"/>
+    <origin xyz="0.386 0.241 -0.25751" rpy="0 0 0"/>
     <geometry>
       <mesh filename="package://ustbot_description/meshes/lidar_back.STL" scale="0.001 0.001 0.001"/>
@@ -313,5 +313,5 @@
 </joint>
 <joint name="lidar_front_joint" type="fixed">
-  <origin xyz="0.386 0.241 0.23751" rpy="0 0 0"/>
+  <origin xyz="0.386 0.241 0.25751" rpy="0 0 0"/>
   <parent link="base_link"/>
   <child link="lidar_front"/>
@@ -319,5 +319,5 @@
 </joint>
 <joint name="lidar_back_joint" type="fixed">
-  <origin xyz="-0.386 -0.241 0.23751" rpy="0 0 0"/>
+  <origin xyz="-0.386 -0.241 0.25751" rpy="0 0 0"/>
   <parent link="base_link"/>
   <child link="lidar_back"/>
