Commit message: Fixing urdf file, fixing map, now global and local costmap can be seen

File: src/Simulation/Descriptions/ustbot_description/urdf/ustbot.gazebo.xacro (robot description, xacro)
@@ -1,4 +1,4 @@
 <?xml version="1.0" ?>
-<robot name="ustbot_sim" xmlns:xacro="http://www.ros.org/wiki/xacro" >
+<robot name="ustbot" xmlns:xacro="http://www.ros.org/wiki/xacro" >
   <xacro:arg name="laser_visual" default="false"/>
   <xacro:property name="body_color" value="Gazebo/Silver" />
@@ -27,5 +27,5 @@
   <!-- *********** simulated ray sensor FRONT side *********** -->
   <gazebo reference="lidar_front">
-    <material>Gazebo/FlatBlack</material>
+    <material>Gazebo/Blue</material>
     <sensor type="ray" name="lidar_front_sensor">
       <pose>0 0 0 0 0 0</pose>
@@ -60,5 +60,5 @@
   <!-- *********** simulated ray sensor BACK side *********** -->
   <gazebo reference="lidar_back">
-    <material>Gazebo/FlatBlack</material>
+    <material>Gazebo/Blue</material>
     <sensor type="ray" name="lidar_back_sensor">
       <pose>0 0 0 0 0 0</pose>
@@ -107,12 +107,4 @@
     <mu1>3500</mu1>
     <mu2>3500</mu2>
-    <selfCollide>true</selfCollide>
-  </gazebo>
-  <gazebo reference="lidar_front">
-    <material>Gazebo/Blue</material>
-    <selfCollide>true</selfCollide>
-  </gazebo>
-  <gazebo reference="lidar_back">
-    <material>Gazebo/Blue</material>
     <selfCollide>true</selfCollide>
   </gazebo>
